File: Hardware/SparkFun_Qwiic_pHAT_Extension.sch (EAGLE design)
At the start: 16 parts, among them J1 RASPBERRYPI-40-PIN-GPIO_SMD_M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, J2 RASPBERRYPI-40-PIN-GPIO_RIGHT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, J3 QWIIC_RIGHT_ANGLE, J5 QWIIC_RIGHT_ANGLE

Commit message: Fixes PWM net names, fixes measures to account for moved stand offs
Connections:
- net 12/PCM0 renamed 12/PWM0
- net 13/PCM1 renamed 13/PWM1
Changed lines of the file:
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@@
 </segment>
 </net>
-<net name="12/PCM0" class="0">
+<net name="12/PWM0" class="0">
 <segment>
 <pinref part="J1" gate="G$1" pin="PWM0/GP12"/>
@@
 </segment>
 </net>
-<net name="13/PCM1" class="0">
+<net name="13/PWM1" class="0">
 <segment>
 <pinref part="J1" gate="G$1" pin="PWM1/GP13"/>
